File: z80-cmos-nmos-tester.kicad_sch (KiCad schematic)
At the start: 41 parts, among them J1 Barrel_Jack, J2 Conn_02x05_Odd_Even, SW1 RESET, SW2 SW_DPDT_x2, U1 Z80CPU, U2 74LS193, U3 74LS02, U4 27C512, U5 74LS573, X1 20MHz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

Commit message: Add CSV BOM and PDF schematic
Other:
- company: (none) -> Chris Tersteeg
- title: (none) -> Z80 CMOS NMOS Tester
Changed lines of the file:
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@@
 (kicad_sch (version 20230121) (generator eeschema)
   (paper "A4")
+  (title_block
+    (title "Z80 CMOS NMOS Tester")
+    (date "2023-9-25")
+    (rev "1.0")
+    (company "Chris Tersteeg")
+  )
   (junction (at 123.19 158.75) (diameter 0) (color 0 0 0 0)
   )
